Commit message: changed gripper urdf to use .stl models

File: cpp/vtk_experiments/gripper_render/hands/franka_gripper/franka_gripper.urdf (robot description, URDF)
Before this commit: robot hand, 5 links, 4 joints
Links:
- link panda_hand: geometry collision cylinder length=0.1 radius=0.07; collision sphere radius=0.07
- link panda_leftfinger: geometry visual mesh filename=meshes/visual/finger.stl
- link panda_rightfinger: geometry visual mesh filename=meshes/visual/finger.stl

Commit message: removed ghost link

File: cpp/vtk_experiments/gripper_render/hands/franka_gripper/franka_gripper.urdf (robot description, URDF)
Before this commit: robot hand, 5 links, 4 joints
Links:
- removed link panda_tcp_fake
Joints:
- removed joint panda_tcp_joint_fake
